Commit message: Future: Combind scan to display.launch

File: src/robot_description/urdf/bb_bot.urdf.xacro (robot description, xacro)
@@ -3,4 +3,7 @@
     <material name="white">
             <color rgba="1 1 1 1"/>
+    </material>
+    <material name="red">
+        <color rgba="1 0 0 1"/>
     </material>
     <material name="black">
@@ -112,3 +115,24 @@
         <axis xyz="0 0 0" />
      </joint>
+     <link name="laser">
+        <visual>
+            <origin xyz="0 0 0" rpy="0 0 0"/>
+            <geometry>
+                <cylinder length="0.0182" radius="0.0255"/>
+            </geometry>
+            <material name="black"/>
+        </visual>
+        <collision>
+            <origin xyz="0 0 0" rpy="0 0 0"/>
+            <geometry>
+                <cylinder length="0.0182" radius="0.0255"/>
+            </geometry>
+        </collision>
+     </link>
+     <joint name="laser_joint" type="fixed">
+        <parent link="base_link"/>
+        <child link="laser" />
+        <origin xyz="0.0925 0 0.0791" rpy="0 0 3.14"/>
+        <axis xyz="0 0 0" />
+     </joint>
 </robot>

Commit message: feture: add robot_bringup

File: src/robot_description/urdf/bb_bot.urdf.xacro (robot description, xacro)
@@ -136,3 +136,18 @@
         <axis xyz="0 0 0" />
      </joint>
+     <link name="imu_frame">
+        <visual>
+            <origin xyz="0 0 0" rpy="0 0 0"/>
+            <geometry>
+                <box size="0.003 0.005 0.002"/>
+            </geometry>
+            <material name="red"/>
+        </visual>
+     </link>
+     <joint name="imu_joint" type="fixed">
+        <parent link="base_link"/>
+        <child link="imu_frame" />
+        <origin xyz="-0.0175 0.05 0.048" rpy="0 0 3.14"/>
+        <axis xyz="0 0 0" />
+     </joint>
 </robot>

Commit message: feature: add nav2, ultrasonics ranger, bumper sensor

File: src/robot_description/urdf/bb_bot.urdf.xacro (robot description, xacro)
@@ -151,3 +151,48 @@
         <axis xyz="0 0 0" />
      </joint>
+     <link name="ranger_center_frame">
+        <visual>
+            <origin xyz="0 0 0" rpy="0 0 0"/>
+            <geometry>
+                <box size="0.015 0.04 0.025"/>
+            </geometry>
+            <material name="black"/>
+        </visual>
+     </link>
+     <joint name="ranger_center_joint" type="fixed">
+        <parent link="base_link"/>
+        <child link="ranger_center_frame" />
+        <origin xyz="0.1725 0 0.01" rpy="0 0 0"/>
+        <axis xyz="0 0 0" />
+     </joint>
+     <link name="ranger_left_frame">
+        <visual>
+            <origin xyz="0 0 0" rpy="0 0 0"/>
+            <geometry>
+                <box size="0.015 0.04 0.025"/>
+            </geometry>
+            <material name="black"/>
+        </visual>
+     </link>
+     <joint name="ranger_left_joint" type="fixed">
+        <parent link="base_link"/>
+        <child link="ranger_left_frame" />
+        <origin xyz="0.1625 0.08 0.01" rpy="0 0 0.6106"/>
+        <axis xyz="0 0 0" />
+     </joint>
+     <link name="ranger_right_frame">
+        <visual>
+            <origin xyz="0 0 0" rpy="0 0 0"/>
+            <geometry>
+                <box size="0.015 0.04 0.025"/>
+            </geometry>
+            <material name="black"/>
+        </visual>
+     </link>
+     <joint name="ranger_right_joint" type="fixed">
+        <parent link="base_link"/>
+        <child link="ranger_right_frame" />
+        <origin xyz="0.1625 -0.08 0.01" rpy="0 0 -0.6106"/>
+        <axis xyz="0 0 0" />
+     </joint>
 </robot>

Commit message: feature: collision monitor

File: src/robot_description/urdf/bb_bot.urdf.xacro (robot description, xacro)
@@ -196,3 +196,18 @@
         <axis xyz="0 0 0" />
      </joint>
+     <link name="camera">
+        <visual>
+            <origin xyz="0 0 0" rpy="0 0 0"/>
+            <geometry>
+                <box size="0.02 0.07 0.03"/>
+            </geometry>
+            <material name="black"/>
+        </visual>
+     </link>
+     <joint name="camerajoint" type="fixed">
+        <parent link="base_link"/>
+        <child link="camera" />
+        <origin xyz="0.1475 0.0 0.055" rpy="0 0 0"/>
+        <axis xyz="0 0 0" />
+     </joint>
 </robot>
