Commit message: Initial commit

File: install/robot_description/share/robot_description/urdf/bb_bot.urdf.xacro (robot description, xacro)
@@ -1,4 +1,5 @@
 <?xml version="1.0"?>
 <robot name="bumperbot" xmlns:xacro="http://ros.org/wiki/xacro">
+<<<<<<< HEAD
     <link name="base_footprint"/>
      <link name="base_link">
@@ -7,4 +8,21 @@
             <box size="0.345 0.2 0.14"/>
         </geometry>
+=======
+    <material name="white">
+            <color rgba="1 1 1 1"/>
+    </material>
+    <material name="black">
+        <color rgba="0 0 0 1"/>
+    </material>
+    <link name="base_footprint"/>
+     <link name="base_link">
+        <visual>
+            <origin xyz="0 0 0" rpy="0 0 0"/>
+            <geometry>
+                <box size="0.345 0.2 0.14"/>
+            </geometry>
+            <material name="white"/>
+        </visual>
+>>>>>>> 267328f (Initial commit)
         <collision>
             <origin xyz="0 0 0" rpy="0 0 0"/>
@@ -17,5 +35,94 @@
         <parent link="base_footprint"/>
         <child link="base_link" />
+<<<<<<< HEAD
         <origin xyz="0 0 0" rpy="0 0 0"/>
       </joint>
+=======
+        <origin xyz="0 0 0.1085" rpy="0 0 0"/>
+     </joint>
+      <link name="right_wheel_link">
+        <visual>
+            <origin xyz="0 0 0" rpy="1.57 0 0"/>
+            <geometry>
+                <cylinder length="0.0254" radius="0.0635"/>
+            </geometry>
+            <material name="black"/>
+        </visual>
+        <collision>
+            <origin xyz="0 0 0" rpy="0 0 0"/>
+            <geometry>
+                <cylinder length="0.0254" radius="0.0635"/>
+            </geometry>
+        </collision>
+      </link>
+      <joint name="right_wheel_joint" type="continuous">
+        <parent link="base_link"/>
+        <child link="right_wheel_link" />
+        <origin xyz="0.0725 -0.11 -0.045" rpy="0 0 0"/>
+        <axis xyz="0 1 0" />
+     </joint>
+     <link name="left_wheel_link">
+        <visual>
+            <origin xyz="0 0 0" rpy="-1.57 0 0"/>
+            <geometry>
+                <cylinder length="0.0254" radius="0.0635"/>
+            </geometry>
+            <material name="black"/>
+        </visual>
+        <collision>
+            <origin xyz="0 0 0" rpy="0 0 0"/>
+            <geometry>
+                <cylinder length="0.0254" radius="0.0635"/>
+            </geometry>
+        </collision>
+      </link>
+      <joint name="left_wheel_joint" type="continuous">
+        <parent link="base_link"/>
+        <child link="left_wheel_link" />
+        <origin xyz="0.0725 0.11 -0.045" rpy="0 0 0"/>
+        <axis xyz="0 1 0" />
+     </joint>
+     <link name="right_caster_link">
+        <visual>
+            <origin xyz="0 0 0" rpy="0 0 0"/>
+            <geometry>
+                <sphere radius="0.0385"/>
+            </geometry>
+            <material name="black"/>
+        </visual>
+        <collision>
+            <origin xyz="0 0 0" rpy="0 0 0"/>
+            <geometry>
+                <sphere radius="0.0385"/>
+            </geometry>
+        </collision>
+     </link>
+     <joint name="right_caster_joint" type="fixed">
+        <parent link="base_link"/>
+        <child link="right_caster_link" />
+        <origin xyz="-0.1125 -0.07 -0.07" rpy="0 0 0"/>
+        <axis xyz="0 0 0" />
+     </joint>
+     <link name="left_caster_link">
+        <visual>
+            <origin xyz="0 0 0" rpy="0 0 0"/>
+            <geometry>
+                <sphere radius="0.0385"/>
+            </geometry>
+            <material name="black"/>
+        </visual>
+        <collision>
+            <origin xyz="0 0 0" rpy="0 0 0"/>
+            <geometry>
+                <sphere radius="0.0385"/>
+            </geometry>
+        </collision>
+     </link>
+     <joint name="left_caster_joint" type="fixed">
+        <parent link="base_link"/>
+        <child link="left_caster_link" />
+        <origin xyz="-0.1125 0.07 -0.07" rpy="0 0 0"/>
+        <axis xyz="0 0 0" />
+     </joint>
+>>>>>>> 267328f (Initial commit)
 </robot>

Commit message: fix file

File: install/robot_description/share/robot_description/urdf/bb_bot.urdf.xacro (robot description, xacro)
@@ -1,12 +1,4 @@
 <?xml version="1.0"?>
 <robot name="bumperbot" xmlns:xacro="http://ros.org/wiki/xacro">
-<<<<<<< HEAD
-    <link name="base_footprint"/>
-     <link name="base_link">
-        <origin xyz="0 0 0" rpy="0 0 0"/>
-        <geometry>
-            <box size="0.345 0.2 0.14"/>
-        </geometry>
-=======
     <material name="white">
             <color rgba="1 1 1 1"/>
@@ -24,5 +16,4 @@
             <material name="white"/>
         </visual>
->>>>>>> 267328f (Initial commit)
         <collision>
             <origin xyz="0 0 0" rpy="0 0 0"/>
@@ -35,8 +26,4 @@
         <parent link="base_footprint"/>
         <child link="base_link" />
-<<<<<<< HEAD
-        <origin xyz="0 0 0" rpy="0 0 0"/>
-      </joint>
-=======
         <origin xyz="0 0 0.1085" rpy="0 0 0"/>
      </joint>
@@ -125,4 +112,3 @@
         <axis xyz="0 0 0" />
      </joint>
->>>>>>> 267328f (Initial commit)
 </robot>

Commit message: feature: add a line notify behavior plugin

File: install/robot_description/share/robot_description/urdf/bb_bot.urdf.xacro (robot description, xacro)
@@ -1 +1,213 @@
-/home/smr/ros2_self_driving_robot/src/robot_description/urdf/bb_bot.urdf.xacro
+<?xml version="1.0"?>
+<robot name="bumperbot" xmlns:xacro="http://ros.org/wiki/xacro">
+    <material name="white">
+            <color rgba="1 1 1 1"/>
+    </material>
+    <material name="red">
+        <color rgba="1 0 0 1"/>
+    </material>
+    <material name="black">
+        <color rgba="0 0 0 1"/>
+    </material>
+    <link name="base_footprint"/>
+     <link name="base_link">
+        <visual>
+            <origin xyz="0 0 0" rpy="0 0 0"/>
+            <geometry>
+                <box size="0.345 0.2 0.14"/>
+            </geometry>
+            <material name="white"/>
+        </visual>
+        <collision>
+            <origin xyz="0 0 0" rpy="0 0 0"/>
+            <geometry>
+                <box size="0.345 0.2 0.14"/>
+            </geometry>
+        </collision>
+     </link>
+     <joint name="base_joint" type="fixed">
+        <parent link="base_footprint"/>
+        <child link="base_link" />
+        <origin xyz="0 0 0.1085" rpy="0 0 0"/>
+     </joint>
+      <link name="right_wheel_link">
+        <visual>
+            <origin xyz="0 0 0" rpy="1.57 0 0"/>
+            <geometry>
+                <cylinder length="0.0254" radius="0.0635"/>
+            </geometry>
+            <material name="black"/>
+        </visual>
+        <collision>
+            <origin xyz="0 0 0" rpy="0 0 0"/>
+            <geometry>
+                <cylinder length="0.0254" radius="0.0635"/>
+            </geometry>
+        </collision>
+      </link>
+      <joint name="right_wheel_joint" type="continuous">
+        <parent link="base_link"/>
+        <child link="right_wheel_link" />
+        <origin xyz="0.0725 -0.11 -0.045" rpy="0 0 0"/>
+        <axis xyz="0 1 0" />
+     </joint>
+     <link name="left_wheel_link">
+        <visual>
+            <origin xyz="0 0 0" rpy="-1.57 0 0"/>
+            <geometry>
+                <cylinder length="0.0254" radius="0.0635"/>
+            </geometry>
+            <material name="black"/>
+        </visual>
+        <collision>
+            <origin xyz="0 0 0" rpy="0 0 0"/>
+            <geometry>
+                <cylinder length="0.0254" radius="0.0635"/>
+            </geometry>
+        </collision>
+      </link>
+      <joint name="left_wheel_joint" type="continuous">
+        <parent link="base_link"/>
+        <child link="left_wheel_link" />
+        <origin xyz="0.0725 0.11 -0.045" rpy="0 0 0"/>
+        <axis xyz="0 1 0" />
+     </joint>
+     <link name="right_caster_link">
+        <visual>
+            <origin xyz="0 0 0" rpy="0 0 0"/>
+            <geometry>
+                <sphere radius="0.0385"/>
+            </geometry>
+            <material name="black"/>
+        </visual>
+        <collision>
+            <origin xyz="0 0 0" rpy="0 0 0"/>
+            <geometry>
+                <sphere radius="0.0385"/>
+            </geometry>
+        </collision>
+     </link>
+     <joint name="right_caster_joint" type="fixed">
+        <parent link="base_link"/>
+        <child link="right_caster_link" />
+        <origin xyz="-0.1125 -0.07 -0.07" rpy="0 0 0"/>
+        <axis xyz="0 0 0" />
+     </joint>
+     <link name="left_caster_link">
+        <visual>
+            <origin xyz="0 0 0" rpy="0 0 0"/>
+            <geometry>
+                <sphere radius="0.0385"/>
+            </geometry>
+            <material name="black"/>
+        </visual>
+        <collision>
+            <origin xyz="0 0 0" rpy="0 0 0"/>
+            <geometry>
+                <sphere radius="0.0385"/>
+            </geometry>
+        </collision>
+     </link>
+     <joint name="left_caster_joint" type="fixed">
+        <parent link="base_link"/>
+        <child link="left_caster_link" />
+        <origin xyz="-0.1125 0.07 -0.07" rpy="0 0 0"/>
+        <axis xyz="0 0 0" />
+     </joint>
+     <link name="laser">
+        <visual>
+            <origin xyz="0 0 0" rpy="0 0 0"/>
+            <geometry>
+                <cylinder length="0.0182" radius="0.0255"/>
+            </geometry>
+            <material name="black"/>
+        </visual>
+        <collision>
+            <origin xyz="0 0 0" rpy="0 0 0"/>
+            <geometry>
+                <cylinder length="0.0182" radius="0.0255"/>
+            </geometry>
+        </collision>
+     </link>
+     <joint name="laser_joint" type="fixed">
+        <parent link="base_link"/>
+        <child link="laser" />
+        <origin xyz="0.0925 0 0.0791" rpy="0 0 3.14"/>
+        <axis xyz="0 0 0" />
+     </joint>
+     <link name="imu_frame">
+        <visual>
+            <origin xyz="0 0 0" rpy="0 0 0"/>
+            <geometry>
+                <box size="0.003 0.005 0.002"/>
+            </geometry>
+            <material name="red"/>
+        </visual>
+     </link>
+     <joint name="imu_joint" type="fixed">
+        <parent link="base_link"/>
+        <child link="imu_frame" />
+        <origin xyz="-0.0175 0.05 0.048" rpy="0 0 3.14"/>
+        <axis xyz="0 0 0" />
+     </joint>
+     <link name="ranger_center_frame">
+        <visual>
+            <origin xyz="0 0 0" rpy="0 0 0"/>
+            <geometry>
+                <box size="0.015 0.04 0.025"/>
+            </geometry>
+            <material name="black"/>
+        </visual>
+     </link>
+     <joint name="ranger_center_joint" type="fixed">
+        <parent link="base_link"/>
+        <child link="ranger_center_frame" />
+        <origin xyz="0.1725 0 0.01" rpy="0 0 0"/>
+        <axis xyz="0 0 0" />
+     </joint>
+     <link name="ranger_left_frame">
+        <visual>
+            <origin xyz="0 0 0" rpy="0 0 0"/>
+            <geometry>
+                <box size="0.015 0.04 0.025"/>
+            </geometry>
+            <material name="black"/>
+        </visual>
+     </link>
+     <joint name="ranger_left_joint" type="fixed">
+        <parent link="base_link"/>
+        <child link="ranger_left_frame" />
+        <origin xyz="0.1625 0.08 0.01" rpy="0 0 0.6106"/>
+        <axis xyz="0 0 0" />
+     </joint>
+     <link name="ranger_right_frame">
+        <visual>
+            <origin xyz="0 0 0" rpy="0 0 0"/>
+            <geometry>
+                <box size="0.015 0.04 0.025"/>
+            </geometry>
+            <material name="black"/>
+        </visual>
+     </link>
+     <joint name="ranger_right_joint" type="fixed">
+        <parent link="base_link"/>
+        <child link="ranger_right_frame" />
+        <origin xyz="0.1625 -0.08 0.01" rpy="0 0 -0.6106"/>
+        <axis xyz="0 0 0" />
+     </joint>
+     <link name="camera">
+        <visual>
+            <origin xyz="0 0 0" rpy="0 0 0"/>
+            <geometry>
+                <box size="0.02 0.07 0.03"/>
+            </geometry>
+            <material name="black"/>
+        </visual>
+     </link>
+     <joint name="camerajoint" type="fixed">
+        <parent link="base_link"/>
+        <child link="camera" />
+        <origin xyz="0.1475 0.0 0.055" rpy="0 0 0"/>
+        <axis xyz="0 0 0" />
+     </joint>
+</robot>
